Commit message: add scripts

File: submodules/usv_gazebo/urdf/components/wamv_3d_lidar.xacro (robot description, xacro)
@@ -40,5 +40,5 @@
         <origin xyz="0 0 -0.035" rpy="0 0 0"/>
         <geometry>
-          <mesh filename="package://usv_gazebo/models/3d_lidar/mesh/3d_lidar.dae"/>
+          <mesh filename="package://vrx_gazebo/models/3d_lidar/mesh/3d_lidar.dae"/>
         </geometry>
       </visual>

File: submodules/usv_gazebo/urdf/thruster_layouts/wamv_aft_thrusters.xacro (robot description, xacro)
@@ -2,8 +2,8 @@
 <robot xmlns:xacro="http://ros.org/wiki/xacro">
   <xacro:include filename="$(find usv_description)/urdf/thrusters/engine.xacro" />
-  <xacro:engine prefix="left" position="0.7 0.7 0.318237" />
-  <xacro:engine prefix="right" position="0.7 -0.7 0.318237" />
-  <xacro:engine prefix="left1" position="-0.7 0.7 0.318237" />
-  <xacro:engine prefix="right1" position="-0.7 -0.7 0.318237" />
+  <xacro:engine prefix="left_front" position="0.7 0.7 0.318237" />
+  <xacro:engine prefix="right_front" position="0.7 -0.7 0.318237" />
+  <xacro:engine prefix="left_rear" position="-0.7 0.7 0.318237" />
+  <xacro:engine prefix="right_rear" position="-0.7 -0.7 0.318237" />
   <gazebo>
     <plugin name="wamv_gazebo_thrust" filename="libusv_gazebo_thrust_plugin.so">
@@ -12,8 +12,8 @@
       <robotNamespace>${namespace}</robotNamespace>
       <xacro:include filename="$(find usv_gazebo)/urdf/thruster_layouts/wamv_gazebo_thruster_config.xacro" />
-      <xacro:wamv_gazebo_thruster_config name="left" />
-      <xacro:wamv_gazebo_thruster_config name="right" />
-      <xacro:wamv_gazebo_thruster_config name="left1" />
-      <xacro:wamv_gazebo_thruster_config name="right1" />
+      <xacro:wamv_gazebo_thruster_config name="left_front" />
+      <xacro:wamv_gazebo_thruster_config name="right_front" />
+      <xacro:wamv_gazebo_thruster_config name="left_rear" />
+      <xacro:wamv_gazebo_thruster_config name="right_rear" />
     </plugin>
   </gazebo>
