Commit message: add controller

File: usv_description/urdf/thrusters/engine.xacro (robot description, xacro)
@@ -42,5 +42,5 @@
       <parent link="${namespace}/${prefix}_engine_link"/>
       <child link="${namespace}/${prefix}_propeller_link"/>
-      <origin rpy="0 0 0" xyz="-0.278156 0 -0.509371"/>
+      <origin rpy="0 0 0" xyz="0 0 -0.509371"/>
       <limit effort="100" velocity="100" />
       <dynamics friction="0.05" damping="0.05" />

File: usv_gazebo/urdf/dynamics/wamv_gazebo_dynamics_plugin.xacro (robot description, xacro)
@@ -14,13 +14,14 @@
         <nDotR>0.0</nDotR>
         <!-- Linear and quadratic drag -->
-        <xU>51.3</xU>
-        <xUU>72.4</xUU>
-        <yV>40.0</yV>
+        <xU>795.3</xU>
+        <xUU>0.0</xUU>
+        <yV>800.0</yV>
         <yVV>0.0</yVV>
         <zW>500.0</zW>
         <kP>50.0</kP>
         <mQ>50.0</mQ>
-        <nR>400.0</nR>
+        <nR>100.0</nR>
         <nRR>0.0</nRR>
+        <!-- mejorar aqui -->
         <!-- General dimensions -->
         <!--<boatArea>2.2</boatArea>-->
