Commit message: modify inertia

File: usv_description/urdf/wamv_base.urdf.xacro (robot description, xacro)
@@ -59,6 +59,6 @@
     </visual-->
     <inertial>
-      <mass value="20.0"/>
-      <inertia ixx="120.0" ixy="0.0" ixz="0.0" iyy="120" iyz="0.0" izz="446.0"/>
+      <mass value="24.0"/>
+      <inertia ixx="120.0" ixy="0.0" ixz="0.0" iyy="125.0" iyz="0.0" izz="120.0"/>
       <!--inertia ixx="120.0" ixy="0.0" ixz="0.0" iyy="393" iyz="0.0" izz="446.0"/-->
     </inertial>

File: usv_gazebo/urdf/dynamics/wamv_gazebo_dynamics_plugin.xacro (robot description, xacro)
@@ -14,13 +14,13 @@
         <nDotR>0.0</nDotR>
         <!-- Linear and quadratic drag -->
-        <xU>795.3</xU>
+        <xU>380.0</xU>
         <xUU>0.0</xUU>
-        <yV>800.0</yV>
+        <yV>400.0</yV>
         <yVV>0.0</yVV>
-        <zW>500.0</zW>
+        <zW>600.0</zW>
         <kP>50.0</kP>
         <mQ>50.0</mQ>
         <nR>100.0</nR>
-        <nRR>0.0</nRR>
+        <nRR>10.0</nRR>
         <!-- mejorar aqui -->
         <!-- General dimensions -->

File: usv_gazebo/urdf/thruster_layouts/wamv_gazebo_thruster_config.xacro (robot description, xacro)
@@ -13,6 +13,6 @@
       <mappingType>1</mappingType>
       <maxCmd>1.0</maxCmd>
-      <maxForceFwd>600.0</maxForceFwd>
-      <maxForceRev>-600.0</maxForceRev>
+      <maxForceFwd>200.0</maxForceFwd>
+      <maxForceRev>-200.0</maxForceRev>
       <!-- modifica fuerza propulsor-->
       <maxAngle>${pi/2}</maxAngle>
