Commit message: modify

File: usv_description/urdf/wamv_base.urdf.xacro (robot description, xacro)
@@ -60,5 +60,6 @@
     <inertial>
       <mass value="24.0"/>
-      <inertia ixx="120.0" ixy="0.0" ixz="0.0" iyy="125.0" iyz="0.0" izz="120.0"/>
+      <inertia ixx="13.76" ixy="0.0" ixz="0.0" iyy="13.76" iyz="0.0" izz="14.45"/>
+            <!--inertia ixx="120.0" ixy="0.0" ixz="0.0" iyy="125.0" iyz="0.0" izz="120.0"/-->
       <!--inertia ixx="120.0" ixy="0.0" ixz="0.0" iyy="393" iyz="0.0" izz="446.0"/-->
     </inertial>

File: usv_gazebo/urdf/dynamics/wamv_gazebo_dynamics_plugin.xacro (robot description, xacro)
@@ -9,10 +9,19 @@
         <waterLevel>0</waterLevel>
         <waterDensity>997.8</waterDensity>
-        <!-- Added mass -->
+ <!-- Added mass -->
         <xDotU>0.0</xDotU>
         <yDotV>0.0</yDotV>
         <nDotR>0.0</nDotR>
         <!-- Linear and quadratic drag -->
-        <xU>200.0</xU>
+        <xU>50.0</xU>
+        <xUU>0.0</xUU>
+        <yV>100.0</yV>
+        <yVV>25.0</yVV>
+        <zW>300.0</zW>
+        <kP>15.0</kP>
+        <mQ>15.0</mQ>
+        <nR>25.0</nR>
+        <nRR>2.5</nRR>
+        <!--xU>200.0</xU>
         <xUU>0.0</xUU>
         <yV>400.0</yV>
@@ -22,12 +31,9 @@
         <mQ>50.0</mQ>
         <nR>100.0</nR>
-        <nRR>10.0</nRR>
-        <!-- mejorar aqui -->
-        <!-- General dimensions -->
-        <!--<boatArea>2.2</boatArea>-->
-        <hullRadius>0.213</hullRadius>
-        <boatWidth>${width}</boatWidth>
+        <nRR>10.0</nRR-->
+    <hullRadius>0.25</hullRadius>
+<boatWidth>${width}</boatWidth>
         <boatLength>${length}</boatLength>
-        <!-- Length discretization, AKA, "N" -->
+    <boatHeight>0.117</boatHeight>
         <length_n>2</length_n>
         <!-- Wave model -->

File: usv_gazebo/urdf/thruster_layouts/wamv_gazebo_thruster_config.xacro (robot description, xacro)
@@ -13,6 +13,6 @@
       <mappingType>1</mappingType>
       <maxCmd>1.0</maxCmd>
-      <maxForceFwd>200.0</maxForceFwd>
-      <maxForceRev>-200.0</maxForceRev>
+      <maxForceFwd>40.0</maxForceFwd>
+      <maxForceRev>-40.0</maxForceRev>
       <!-- modifica fuerza propulsor-->
       <maxAngle>${pi/2}</maxAngle>

Commit message: modify velocity controller

File: usv_description/urdf/wamv_base.urdf.xacro (robot description, xacro)
@@ -60,5 +60,6 @@
     <inertial>
       <mass value="24.0"/>
-      <inertia ixx="13.76" ixy="0.0" ixz="0.0" iyy="13.76" iyz="0.0" izz="14.45"/>
+      <!--inertia ixx="13.76" ixy="0.0" ixz="0.0" iyy="13.76" iyz="0.0" izz="14.45"/-->
+      <inertia ixx="4.77" ixy="0.0" ixz="0.0" iyy="1.01" iyz="0.0" izz="5.78"/>
             <!--inertia ixx="120.0" ixy="0.0" ixz="0.0" iyy="125.0" iyz="0.0" izz="120.0"/-->
       <!--inertia ixx="120.0" ixy="0.0" ixz="0.0" iyy="393" iyz="0.0" izz="446.0"/-->

File: usv_gazebo/urdf/dynamics/wamv_gazebo_dynamics_plugin.xacro (robot description, xacro)
@@ -14,13 +14,15 @@
         <nDotR>0.0</nDotR>
         <!-- Linear and quadratic drag -->
-        <xU>50.0</xU>
-        <xUU>0.0</xUU>
-        <yV>100.0</yV>
-        <yVV>25.0</yVV>
-        <zW>300.0</zW>
-        <kP>15.0</kP>
-        <mQ>15.0</mQ>
-        <nR>25.0</nR>
-        <nRR>2.5</nRR>
+        <xU>23.0</xU>
+        <xUU>38.0</xUU>
+        <yV>40.0</yV>
+        <yVV>30.0</yVV>
+        <zW>500.0</zW>
+        <kP>100.0</kP>
+        <kPP>100.0</kPP>
+        <mQ>100.0</mQ>
+        <mQQ>100.0</mQQ>
+        <nR>100.0</nR>
+        <nRR>10.0</nRR>
         <!--xU>200.0</xU>
         <xUU>0.0</xUU>
