Commit message: add data

File: usv_gazebo/urdf/components/lidar.xacro (robot description, xacro)
@@ -14,6 +14,4 @@
                            post_Y="${post_Y}" post_z_from="${post_z_from}"
                            vertical_lasers="16"/>
-      <!--specs for 16 beam lidar are implemented by default.
-          See wamv_3d_lidar for those-->
     </xacro:if>
     <xacro:if value="${type == '32_beam'}">

File: usv_gazebo/urdf/components/wamv_3d_lidar copy.xacro (robot description, xacro)
@@ -1,11 +1,24 @@
 <?xml version="1.0" encoding="UTF-8"?>
 <robot xmlns:xacro="http://ros.org/wiki/xacro">
-  <!-- Macro 3D LIDAR (aprox Livox Mid-360) usando el MISMO plugin gpu_ray + gazebo_ros_velodyne_gpu_laser -->
-  <!-- Cambios clave por defecto:
-       - 360° horizontales    : min_angle = -pi, max_angle = +pi
-       - FOV vertical ~60°     : -20° .. +40°
-       - Densidad moderada     : samples=3600 (≈0.1°) y vertical_lasers=6
-       - Rango y ruido         : max_range=70 m, noise_stddev=0.002
-       - update_rate           : 20 Hz (ajustable)
+  <!-- Macro to insert a 3D scanning LIDAR with ROS integration
+    name: Prefix used for naming.
+    x: X position of the laser (from the base_link).
+    y: Y position of the laser (from the base_link).
+    z: Z position of the laser (from the base_link).
+    R: Roll orientation of the laser (from the laser's origin).
+    P: Pitch orientation of the laser (from the laser's origin).
+    Y: Yaw orientation of the laser (from the laser's origin).
+    post_Y: Yaw orientation of the post (from the post's origin).
+    post_z_from: Z position of the post's base.
+    update_rate: frequency to publish output, hz
+    vertical_lasers: number of vertical lasers which spin about Z to generate output
+    samples: number of samples during spin, higher is more dense but slows down simulation
+    resolution: This number is multiplied by samples to determine the number of range data points returned.
+    min_angle: the horizontal angle that the scan begins at
+    max_angle: the angle that the scan ends at
+    min_vertical_angle: the angle of the lowest vertical beam
+    max_vertical_angle: the angle of the highest vertical beam
+    max_range: maximum distance for an object to be detected by laser
+    noise_stddev: Standard deviation of gaussian noise applied to output pointcloud
   -->
   <xacro:macro name="wamv_3d_lidar" params="name
@@ -13,20 +26,14 @@
                                             R:=0 P:=0 Y:=0
                                             post_Y:=0 post_z_from:=1.2965
-                                            update_rate:=20
-                                            vertical_lasers:=6
-                                            samples:=3600
-                                            resolution:=1
-                                            min_angle:=${-pi}
-                                            max_angle:=${pi}
-                                            min_vertical_angle:=${radians(-20)}
-                                            max_vertical_angle:=${radians(40)}
-                                            max_range:=70
-                                            noise_stddev:=0.002">
-    <!-- Posicionamiento mecánico -->
+                                            update_rate:=10 vertical_lasers:=16 samples:=1875 resolution:=0.1
+                                            min_angle:=${-3*pi/4} max_angle:=${3*pi/4}
+                                            min_vertical_angle:=${-pi/12} max_vertical_angle:=${pi/12}
+                                            max_range:=200 noise_stddev:=0.001">
+    <!-- Define length variables for link positioning -->
     <xacro:property name="platform_z" value="${post_z_from}"/>
     <xacro:property name="post_to_post_arm_x" value="0.03"/>
     <xacro:property name="post_arm_to_lidar_x" value="0.04"/>
     <xacro:property name="post_arm_to_lidar_z" value="0.05"/>
-    <!-- Link del sensor -->
+    <!-- 3d lidar sensor -->
     <link name="${namespace}/${name}_link">
       <visual name="${name}_visual">
@@ -43,19 +50,32 @@
       <inertial>
         <mass value="1"/>
-        <inertia ixx="0.00109375" iyy="0.00109375" izz="0.00125" ixy="0" ixz="0" iyz="0"/>
+        <inertia
+          ixx="0.00109375"
+          iyy="0.00109375"
+          izz="0.00125"
+          ixy="0"
+          ixz="0"
+          iyz="0"/>
       </inertial>
     </link>
-    <!-- Post del sensor -->
+    <!-- Define post length and mass based on desired z position of sensor -->
     <xacro:property name="post_length" value="${z-platform_z-post_arm_to_lidar_z}"/>
     <xacro:property name="post_mass_per_meter" value="0.9"/>
     <xacro:property name="post_mass" value="${post_mass_per_meter * post_length}"/>
     <xacro:property name="post_radius" value="0.0076"/>
+    <!-- Sensor post -->
     <link name="${namespace}/${name}_post_link">
       <visual>
-        <geometry><cylinder radius="${post_radius}" length="${post_length}"/></geometry>
-        <material name="${name}_post_material"><color rgba="0.0 0.0 0.0 1.0"/></material>
+        <geometry>
+          <cylinder radius="${post_radius}" length="${post_length}"/>
+        </geometry>
+        <material name="${name}_post_material">
+          <color rgba="0.0 0.0 0.0 1.0"/>
+        </material>
       </visual>
       <collision name="${name}_post_collision">
-        <geometry><cylinder radius="${post_radius}" length="${post_length}"/></geometry>
+        <geometry>
+          <cylinder radius="${post_radius}" length="${post_length}"/>
+        </geometry>
       </collision>
       <inertial>
@@ -65,8 +85,10 @@
           iyy="${(post_mass/12) * (3*post_radius*post_radius + post_length*post_length)}"
           izz="${(post_mass/2) * (post_radius*post_radius)}"
-          ixy="0" ixz="0" iyz="0"/>
+          ixy="0"
+          ixz="0"
+          iyz="0"/>
       </inertial>
     </link>
-    <!-- Brazo del post -->
+    <!-- Sensor post arm -->
     <link name="${namespace}/${name}_post_arm_link">
       <visual name="${name}_post_arm_visual">
@@ -78,31 +100,40 @@
       <collision name="${name}_post_arm_collision">
         <origin xyz="0 0 0" rpy="${radians(-60)-pi/20} 0 ${-pi/2}"/>
-        <geometry><cylinder radius="0.008" length="0.065"/></geometry>
+        <geometry>
+          <cylinder radius="0.008" length="0.065"/>
+        </geometry>
       </collision>
       <inertial>
         <origin xyz="0 0 0" rpy="${radians(-60)-pi/20} 0 ${-pi/2}"/>
         <mass value="0.1"/>
-        <inertia ixx="0.00003680833" iyy="0.00003680833" izz="0.0000032" ixy="0" ixz="0" iyz="0"/>
+        <inertia
+          ixx="0.00003680833"
+          iyy="0.00003680833"
+          izz="0.00000320000"
+          ixy="0"
+          ixz="0"
+          iyz="0"/>
       </inertial>
     </link>
-    <!-- Juntas fijas -->
+    <!-- Base to sensor post joint -->
     <xacro:property name="post_z" value="${platform_z+post_length/2}"/>
     <xacro:property name="post_to_lidar_x" value="${post_to_post_arm_x+post_arm_to_lidar_x}"/>
     <joint name="${namespace}/base_to_${name}_post_joint" type="fixed">
-      <origin xyz="${x-(post_to_lidar_x)*cos(post_Y)} ${y-(post_to_lidar_x)*sin(post_Y)} ${post_z}" rpy="0 0 ${post_Y}"/>
-      <parent link="${namespace}/base_link"/>
-      <child  link="${namespace}/${name}_post_link"/>
+      <origin xyz="${x-(post_to_lidar_x)*cos(post_Y)} ${y-(post_to_lidar_x)*sin(post_Y)} ${post_z}" rpy="0 0 ${post_Y}" />
+      <parent link="${namespace}/base_link" />
+      <child link="${namespace}/${name}_post_link" />
     </joint>
+    <!-- Sensor post to sensor post arm joint -->
     <joint name="${namespace}/${name}_post_to_${name}_post_arm_joint" type="fixed">
-      <origin xyz="${post_to_post_arm_x} 0 ${z-post_z-post_arm_to_lidar_z}" rpy="0 0 0"/>
-      <parent link="${namespace}/${name}_post_link"/>
-      <child  link="${namespace}/${name}_post_arm_link"/>
+      <origin xyz="${post_to_post_arm_x} 0 ${z-post_z-post_arm_to_lidar_z}" rpy="0 0 0" />
+      <parent link="${namespace}/${name}_post_link" />
+      <child link="${namespace}/${name}_post_arm_link" />
     </joint>
+    <!-- Sensor post arm to lidar joint -->
     <joint name="${namespace}/${name}_post_arm_to_${name}_joint" type="fixed">
-      <origin xyz="${post_arm_to_lidar_x} 0 ${post_arm_to_lidar_z}" rpy="${R} ${P} ${Y-post_Y}"/>
-      <parent link="${namespace}/${name}_post_arm_link"/>
-      <child  link="${namespace}/${name}_link"/>
+      <origin xyz="${post_arm_to_lidar_x} 0 ${post_arm_to_lidar_z}" rpy="${R} ${P} ${Y-post_Y}" />
+      <parent link="${namespace}/${name}_post_arm_link" />
+      <child link="${namespace}/${name}_link" />
     </joint>
-    <!-- Sensor GPU (Velodyne) configurado para emular Livox 360 -->
     <gazebo reference="${namespace}/${name}_link">
       <sensor type="gpu_ray" name="${name}_sensor">
@@ -111,5 +142,4 @@
           <scan>
             <horizontal>
-              <!-- 360° completos -->
               <samples>${samples/resolution}</samples>
               <resolution>${resolution}</resolution>
@@ -118,5 +148,4 @@
             </horizontal>
             <vertical>
-              <!-- Pocas “capas” para no parecer multi-anillo clásico -->
               <samples>${vertical_lasers}</samples>
               <resolution>1</resolution>
@@ -135,17 +164,12 @@
           </noise>
         </ray>
-        <!-- Plugin ROS que publica PointCloud2 -->
         <plugin name="${name}_plugin" filename="libgazebo_ros_velodyne_gpu_laser.so">
           <topicName>${namespace}/${sensor_namespace}lidars/${name}/points</topicName>
           <frameName>${namespace}/${name}_link</frameName>
           <min_intensity>0</min_intensity>
-          <!-- Opcionales (si tu build los soporta):
-          <organize_cloud>false</organize_cloud>
-          <skip>0</skip>
-          -->
         </plugin>
       </sensor>
     </gazebo>
-    <!-- Material del post -->
+    <!-- Set color of post -->
     <gazebo reference="${namespace}/${name}_post_link">
       <material>Gazebo/Black</material>

File: usv_gazebo/urdf/components/wamv_gps.xacro (robot description, xacro)
@@ -27,11 +27,9 @@
       </inertial>
     </link>
-    <joint name="${namespace}/${name}_joint" type="revolute">
-      <axis xyz="0 0 1"/>
-      <limit effort="1000.0" lower="0.0" upper="0" velocity="0"/>
-      <origin xyz="${x} ${y} ${z}" rpy="${R} ${P} ${Y}" />
-      <parent link="${namespace}/base_link" />
-      <child link="${namespace}/${name}_link" />
-    </joint>
+<joint name="${namespace}/${name}_joint" type="fixed">
+  <origin xyz="${x} ${y} ${z}" rpy="${R} ${P} ${Y}" />
+  <parent link="${namespace}/base_link" />
+  <child link="${namespace}/${name}_link" />
+</joint>
     <gazebo>
       <plugin name="gps_plugin_${name}" filename="libhector_gazebo_ros_gps.so">

File: usv_gazebo/urdf/components/wamv_imu.xacro (robot description, xacro)
@@ -8,5 +8,6 @@
         </geometry>
         <material name="${name}_visual_material">
-          <color rgba="1.0 0.0 00 1.0" />
+          <!-- corrige el color (era '00') -->
+          <color rgba="1.0 0.0 0.0 1.0" />
         </material>
       </visual>
@@ -16,7 +17,7 @@
       </inertial>
     </link>
-    <joint name="${namespace}/${name}_joint" type="revolute">
-      <axis xyz="0 0 1"/>
-      <limit effort="1000.0" lower="0.0" upper="0" velocity="0"/>
+    <!-- ANTES: type="revolute" con límites 0..0 -->
+    <!-- AHORA: joint FIXED para que robot_state_publisher publique la TF sin joint_states -->
+    <joint name="${namespace}/${name}_joint" type="fixed">
       <origin xyz="${x} ${y} ${z}" rpy="${R} ${P} ${Y}"/>
       <parent link="${namespace}/base_link"/>
@@ -29,5 +30,4 @@
         <topicName>${namespace}/${sensor_namespace}imu/imu/data</topicName>
         <serviceName>${namespace}/${sensor_namespace}imu_service</serviceName>
-        <!-- Manually prepend namespace to tf frame. -->
         <frameId>${namespace}/${name}_link</frameId>
         <alwaysOn>true</alwaysOn>

File: usv_gazebo/urdf/macros.xacro (robot description, xacro)
@@ -2,8 +2,6 @@
 <!-- Includes all macros in this package so they don't need to be included individualy -->
 <robot xmlns:xacro="http://ros.org/wiki/xacro"
-       name="WAM-V">
-  <!-- Include dynamics macros -->
+       name="iacquabot">
   <xacro:include filename="$(find usv_gazebo)/urdf/dynamics/wamv_gazebo_dynamics_plugin.xacro" />
-  <!-- Include sensor macros -->
   <xacro:include filename="$(find usv_gazebo)/urdf/components/wamv_camera.xacro" />
   <xacro:include filename="$(find usv_gazebo)/urdf/components/wamv_gps.xacro" />
@@ -16,5 +14,4 @@
   <xacro:include filename="$(find usv_gazebo)/urdf/components/wamv_p3d.xacro" />
   <xacro:include filename="$(find usv_gazebo)/urdf/components/wamv_pinger.xacro" />
-  <!-- Include ball shooter macros -->
   <xacro:include filename="$(find usv_gazebo)/urdf/components/ball_shooter.xacro" />
 </robot>

File: usv_gazebo/urdf/wamv_gazebo.urdf.xacro (robot description, xacro)
@@ -2,5 +2,5 @@
 <!-- Basic WAM-V with gazebo plugins for dynamics -->
 <robot xmlns:xacro="http://ros.org/wiki/xacro"
-       name="WAM-V">
+       name="iacquabot">
   <xacro:arg name="locked" default="false" />
   <xacro:arg name="thruster_config" default="H" />
@@ -20,5 +20,5 @@
   <!-- Note: this is only used for some sensors that do not correctly use the
   robotNamespace parameter -->
-  <xacro:arg name="namespace" default="wamv"/>
+  <xacro:arg name="namespace" default="iacquabot"/>
   <xacro:property name="thruster_namespace" value="$(arg thruster_namespace)" scope="global" />
   <xacro:property name="camera_namespace" value="$(arg camera_namespace)" scope="global" />
